File: Util/Ordering Info/AutoPowerBoxTesterv1.1/AutoPBT.brd (EAGLE design)
At the start: 191.8 x 144.8 mm, 98 parts, among them J1 39301039CON_39301039, J10 TB001-500-07BE, J11 430450212CON_430450212_MOL, J2 39281083CON_39281083, J3 39281023CON_39281023, J4 39281123CON_39281123, J5 39281063CON_39281063, J6 39299046CON_39299046, J7 PJ-202AH, J8 TB001-500-07BE, J9 TB001-500-07BE, K1 J107F1CS203VDC.80, U1 LM1086CT-5.0/NOPB, U10 VOL628A-3T, U11 VOL628A-3T, U12 VOL628A-3T, U13 PZTA06SOT-223_ONS, U14 PZTA06SOT-223_ONS, U15 VOL628A-3T, U16 VOL628A-3T, U17 VOL628A-3T, U18 VOL628A-3T, U19 AQY212GHAX, U2 LM1086CT-3.3/NOPB, U20 AQY212GHAX, U21 PZTA06SOT-223_ONS, U22 PZTA06SOT-223_ONS, U23 VOL628A-3T, U24 VOL628A-3T, U25 AQY212GHAX, U26 AQY212GHAX, U27 PZTA06SOT-223_ONS, U28 PZTA06SOT-223_ONS, U29 VOL628A-3T, U3 VOL628A-3T, U30 VOL628A-3T, U4 VOL628A-3T, U5 VOL628A-3T, U6 PZTA06SOT-223_ONS, U7 PZTA06SOT-223_ONS, U8 AQY212GHAX, U9 AQY212GHAX

Commit message: Updated readme and ordering info
Parts:
- C1, C2: device Capacitor:CAPC1608X85 -> Capacitor:CAPC3216X135
- R45, R46: value 100K -> 100k; device Resistor:RESC1608X60 -> Resistor:RESC6332X71
- moved R45 2.84 mm to (-15.2, 22.9), turned to 0 degrees
- moved R46 1.80 mm to (-29.2, 22.9), turned to 0 degrees
Connections:
- removed net N$7: R46.2
Routing:
- net BLOW_P5: track 264.9 -> 262.4 mm
- net N$21: track 11.2 -> 12.8 mm
- net N$42: track 11.1 -> 12.3 mm
